Commit message: adding base go2 urdf

File: resources/go2/urdf/go2.urdf (robot description, URDF)
Before this commit: robot anymal, 67 links, 66 joints
Links:
- removed link FL_calflower
- removed link FL_calflower1
- removed link FR_calflower
- removed link FR_calflower1
- removed link LF_hip
- removed link LF_shank
- removed link LF_thigh
- removed link LH_hip
- removed link LH_shank
- removed link LH_thigh
- removed link RF_hip
- removed link RF_shank
- removed link RF_thigh
- removed link RH_hip
- removed link RH_shank
- removed link RH_thigh
- removed link RL_calflower
- removed link RL_calflower1
- removed link RR_calflower
- removed link RR_calflower1
- added link LF_HAA_drive, mass 2.01511; visual mesh filename=package://ocs2_robotic_assets/resources/anymal_d/meshes/dri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 scale=1.0 1.0 1.0
- added link LF_HFE_drive, mass 2.01511; collision cylinder length=0.119 radius=0.05375; visual mesh filename=package://ocs2_robotic_assets/resources/anymal_d/meshes/dri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 scale=1.0 1.0 1.0
- added link LF_HFE_output, mass 0.001
- added link LF_HIP, mass 0.001
- added link LF_KFE_drive, mass 2.01511; collision cylinder length=0.119 radius=0.05375; visual mesh filename=package://ocs2_robotic_assets/resources/anymal_d/meshes/dri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 scale=1.0 1.0 1.0
- added link LF_SHANK, mass 0.001
- added link LF_THIGH, mass 0.001
- added link LF_hip_fixed, mass 0.36386; visual mesh filename=package://ocs2_robotic_assets/resources/anymal_d/meshes/hip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 scale=1.0 1.0 1.0
- added link LF_shank_fixed, mass 0.49854; collision box size=0.13283 0.08302 0.05732; collision cylinder length=0.05732 radius=0.071
- added link LF_thigh_fixed, mass 1.10098; collision box size=0.093 0.063 0.285; collision cylinder length=0.08313000000000001 radius=0.07
- added link LH_HAA_drive, mass 2.01511; visual mesh filename=package://ocs2_robotic_assets/resources/anymal_d/meshes/dri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 scale=1.0 1.0 1.0
- added link LH_HFE_drive, mass 2.01511; collision cylinder length=0.119 radius=0.05375; visual mesh filename=package://ocs2_robotic_assets/resources/anymal_d/meshes/dri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 scale=1.0 1.0 1.0
- added link LH_HFE_output, mass 0.001
- added link LH_HIP, mass 0.001
- added link LH_KFE_drive, mass 2.01511; collision cylinder length=0.119 radius=0.05375; visual mesh filename=package://ocs2_robotic_assets/resources/anymal_d/meshes/dri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 scale=1.0 1.0 1.0
- added link LH_SHANK, mass 0.001
- added link LH_THIGH, mass 0.001
- added link LH_hip_fixed, mass 0.36386; visual mesh filename=package://ocs2_robotic_assets/resources/anymal_d/meshes/hip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 scale=1.0 1.0 1.0
- added link LH_shank_fixed, mass 0.49854; collision box size=0.13283 0.08302 0.05732; collision cylinder length=0.05732 radius=0.071
- added link LH_thigh_fixed, mass 1.10098; collision box size=0.093 0.063 0.285; collision cylinder length=0.08313000000000001 radius=0.07
- added link RF_HAA_drive, mass 2.01511; visual mesh filename=package://ocs2_robotic_assets/resources/anymal_d/meshes/dri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 scale=1.0 1.0 1.0
- added link RF_HFE_drive, mass 2.01511; collision cylinder length=0.119 radius=0.05375; visual mesh filename=package://ocs2_robotic_assets/resources/anymal_d/meshes/dri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 scale=1.0 1.0 1.0
- added link RF_HFE_output, mass 0.001
- added link RF_HIP, mass 0.001
- added link RF_KFE_drive, mass 2.01511; collision cylinder length=0.119 radius=0.05375; visual mesh filename=package://ocs2_robotic_assets/resources/anymal_d/meshes/dri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 scale=1.0 1.0 1.0
- added link RF_SHANK, mass 0.001
- added link RF_THIGH, mass 0.001
- added link RF_hip_fixed, mass 0.36386; visual mesh filename=package://ocs2_robotic_assets/resources/anymal_d/meshes/hip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 scale=1.0 1.0 1.0
- added link RF_shank_fixed, mass 0.49854; collision box size=0.13283 0.08302 0.05732; collision cylinder length=0.05732 radius=0.071
- added link RF_thigh_fixed, mass 1.10098; collision box size=0.093 0.063 0.285; collision cylinder length=0.08313000000000001 radius=0.07
- added link RH_HAA_drive, mass 2.01511; visual mesh filename=package://ocs2_robotic_assets/resources/anymal_d/meshes/dri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 scale=1.0 1.0 1.0
- added link RH_HFE_drive, mass 2.01511; collision cylinder length=0.119 radius=0.05375; visual mesh filename=package://ocs2_robotic_assets/resources/anymal_d/meshes/dri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 scale=1.0 1.0 1.0
- added link RH_HFE_output, mass 0.001
- added link RH_HIP, mass 0.001
- added link RH_KFE_drive, mass 2.01511; collision cylinder length=0.119 radius=0.05375; visual mesh filename=package://ocs2_robotic_assets/resources/anymal_d/meshes/dri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 scale=1.0 1.0 1.0
- added link RH_SHANK, mass 0.001
- added link RH_THIGH, mass 0.001
- added link RH_hip_fixed, mass 0.36386; visual mesh filename=package://ocs2_robotic_assets/resources/anymal_d/meshes/hip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 scale=1.0 1.0 1.0
- added link RH_shank_fixed, mass 0.49854; collision box size=0.13283 0.08302 0.05732; collision cylinder length=0.05732 radius=0.071
- added link RH_thigh_fixed, mass 1.10098; collision box size=0.093 0.063 0.285; collision cylinder length=0.08313000000000001 radius=0.07
- link LF_FOOT: mass 0.04 -> 0.29644; geometry collision cylinder length=0.39572 radius=0.0175; collision sphere radius=0.031455
- link LH_FOOT: mass 0.04 -> 0.29644; geometry collision cylinder length=0.39572 radius=0.0175; collision sphere radius=0.031455
- link RF_FOOT: mass 0.04 -> 0.29644; geometry collision cylinder length=0.39572 radius=0.0175; collision sphere radius=0.031455
- link RH_FOOT: mass 0.04 -> 0.29644; geometry collision cylinder length=0.39572 radius=0.0175; collision sphere radius=0.031455
- link base: mass 6.921 -> None; geometry collision box size=0.894 0.1615 0.256; collision cylinder length=0.1482 radius=0.089
- link battery: geometry visual mesh filename=package://ocs2_robotic_assets/resources/anymal_d/meshes/bat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 scale=1.0 1.0 1.0
- link bottom_shell: geometry visual mesh filename=package://ocs2_robotic_assets/resources/anymal_d/meshes/bot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 scale=1.0 1.0 1.0
- link docking_socket: geometry visual mesh filename=package://ocs2_robotic_assets/resources/anymal_d/meshes/doc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 scale=1.0 1.0 1.0
- link face_shell_front: geometry visual mesh filename=package://ocs2_robotic_assets/resources/anymal_d/meshes/fac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 scale=1.0 1.0 1.0
- link face_shell_rear: geometry visual mesh filename=package://ocs2_robotic_assets/resources/anymal_d/meshes/fac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 scale=1.0 1.0 1.0
- link lidar: geometry collision cylinder length=0.1355 radius=0.07; visual mesh filename=package://ocs2_robotic_assets/resources/anymal_d/meshes/lid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
- link top_shell: geometry visual mesh filename=package://ocs2_robotic_assets/resources/anymal_d/meshes/top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 scale=1.0 1.0 1.0
Joints:
- removed joint FL_calflower1_joint
- removed joint FL_calflower_joint
- removed joint FL_foot_joint
- removed joint FR_calflower1_joint
- removed joint FR_calflower_joint
- removed joint FR_foot_joint
- removed joint RL_calflower1_joint
- removed joint RL_calflower_joint
- removed joint RL_foot_joint
- removed joint RR_calflower1_joint
- removed joint RR_calflower_joint
- removed joint RR_foot_joint
- added joint LF_HFE_drive_LF_thigh_fixed: type fixed, parent LF_HFE_drive, child LF_thigh_fixed, origin xyz=0 0 0 rpy=0 0 1.5707963267948966
- added joint LF_HIP_LF_hip_fixed: type fixed, parent LF_HIP, child LF_hip_fixed, origin xyz=0 0 0 rpy=0 0 0.0
- added joint LF_THIGH_to_LF_HFE_drive: type fixed, parent LF_THIGH, child LF_HFE_drive, origin xyz=0 0 0 rpy=0 0 0
- added joint LF_hip_fixed_LF_HFE_output: type fixed, parent LF_hip_fixed, child LF_HFE_output, origin xyz=0.069 0.006 0.0 rpy=0 0 -1.5707963267948966
- added joint LF_shank_LF_shank_fixed: type fixed, parent LF_SHANK, child LF_shank_fixed, origin xyz=0 0 0 rpy=0 0 -1.5707963267948966
- added joint LF_shank_fixed_LF_FOOT: type fixed, parent LF_shank_fixed, child LF_FOOT, origin xyz=0.1 0.02225 -0.39246 rpy=0 0 0
- added joint LF_thigh_fixed_LF_KFE_drive: type fixed, parent LF_thigh_fixed, child LF_KFE_drive, origin xyz=0.0 0.1805 -0.285 rpy=0 0 1.5707963267948966
- added joint LH_HFE_drive_LH_thigh_fixed: type fixed, parent LH_HFE_drive, child LH_thigh_fixed, origin xyz=0 0 0 rpy=0 0 1.5707963267948966
- added joint LH_HIP_LH_hip_fixed: type fixed, parent LH_HIP, child LH_hip_fixed, origin xyz=0 0 0 rpy=0 0 -3.141592653589793
- added joint LH_THIGH_to_LH_HFE_drive: type fixed, parent LH_THIGH, child LH_HFE_drive, origin xyz=0 0 0 rpy=0 0 0
- added joint LH_hip_fixed_LH_HFE_output: type fixed, parent LH_hip_fixed, child LH_HFE_output, origin xyz=-0.069 0.006 0.0 rpy=0 0 -1.5707963267948966
- added joint LH_shank_LH_shank_fixed: type fixed, parent LH_SHANK, child LH_shank_fixed, origin xyz=0 0 0 rpy=0 0 -1.5707963267948966
- added joint LH_shank_fixed_LH_FOOT: type fixed, parent LH_shank_fixed, child LH_FOOT, origin xyz=-0.1 0.02225 -0.39246 rpy=0 0 0
- added joint LH_thigh_fixed_LH_KFE_drive: type fixed, parent LH_thigh_fixed, child LH_KFE_drive, origin xyz=-0.0 0.1805 -0.285 rpy=0 0 1.5707963267948966
- added joint RF_HFE_drive_RF_thigh_fixed: type fixed, parent RF_HFE_drive, child RF_thigh_fixed, origin xyz=0 0 0 rpy=0 0 -1.5707963267948966
- added joint RF_HIP_RF_hip_fixed: type fixed, parent RF_HIP, child RF_hip_fixed, origin xyz=0 0 0 rpy=0 0 0.0
- added joint RF_THIGH_to_RF_HFE_drive: type fixed, parent RF_THIGH, child RF_HFE_drive, origin xyz=0 0 0 rpy=0 0 0
- added joint RF_hip_fixed_RF_HFE_output: type fixed, parent RF_hip_fixed, child RF_HFE_output, origin xyz=0.069 -0.006 0.0 rpy=0 0 1.5707963267948966
- added joint RF_shank_RF_shank_fixed: type fixed, parent RF_SHANK, child RF_shank_fixed, origin xyz=0 0 0 rpy=0 0 1.5707963267948966
- added joint RF_shank_fixed_RF_FOOT: type fixed, parent RF_shank_fixed, child RF_FOOT, origin xyz=0.1 -0.02225 -0.39246 rpy=0 0 0
- added joint RF_thigh_fixed_RF_KFE_drive: type fixed, parent RF_thigh_fixed, child RF_KFE_drive, origin xyz=0.0 -0.1805 -0.285 rpy=0 0 -1.5707963267948966
- added joint RH_HFE_drive_RH_thigh_fixed: type fixed, parent RH_HFE_drive, child RH_thigh_fixed, origin xyz=0 0 0 rpy=0 0 -1.5707963267948966
- added joint RH_HIP_RH_hip_fixed: type fixed, parent RH_HIP, child RH_hip_fixed, origin xyz=0 0 0 rpy=0 0 -3.141592653589793
- added joint RH_THIGH_to_RH_HFE_drive: type fixed, parent RH_THIGH, child RH_HFE_drive, origin xyz=0 0 0 rpy=0 0 0
- added joint RH_hip_fixed_RH_HFE_output: type fixed, parent RH_hip_fixed, child RH_HFE_output, origin xyz=-0.069 -0.006 0.0 rpy=0 0 1.5707963267948966
- added joint RH_shank_RH_shank_fixed: type fixed, parent RH_SHANK, child RH_shank_fixed, origin xyz=0 0 0 rpy=0 0 1.5707963267948966
- added joint RH_shank_fixed_RH_FOOT: type fixed, parent RH_shank_fixed, child RH_FOOT, origin xyz=-0.1 -0.02225 -0.39246 rpy=0 0 0
- added joint RH_thigh_fixed_RH_KFE_drive: type fixed, parent RH_thigh_fixed, child RH_KFE_drive, origin xyz=-0.0 -0.1805 -0.285 rpy=0 0 -1.5707963267948966
- added joint base_LF_HAA_drive: type fixed, parent base, child LF_HAA_drive, origin xyz=0.304 0.109 0.0 rpy=0 0 0.0
- added joint base_LH_HAA_drive: type fixed, parent base, child LH_HAA_drive, origin xyz=-0.304 0.109 0.0 rpy=0 0 -3.141592653589793
- added joint base_RF_HAA_drive: type fixed, parent base, child RF_HAA_drive, origin xyz=0.304 -0.109 0.0 rpy=0 0 0.0
- added joint base_RH_HAA_drive: type fixed, parent base, child RH_HAA_drive, origin xyz=-0.304 -0.109 0.0 rpy=0 0 -3.141592653589793
- joint LF_HAA: child LF_hip -> LF_HIP; limit lower=-1.0472 upper=1.0472 effort=23.7 velocity=30.1 -> lower=-0.7853985 upper=0.6108655 effort=80.0 velocity=8.5; origin xyz=0.1934 0.0465 0 rpy=0 0 0 -> xyz=0 0 0 rpy=0 0 0; parent base -> LF_HAA_drive
- joint LF_HFE: axis 0 1 0 -> -1 0 0; child LF_thigh -> LF_THIGH; limit lower=-1.5708 upper=3.4907 effort=23.7 velocity=30.1 -> lower=-9.42477796076938 upper=9.42477796076938 effort=80.0 velocity=8.5; origin xyz=0 0.0955 0 rpy=0 0 0 -> xyz=0 0 0 rpy=0 0 0; parent LF_hip -> LF_HFE_output
- joint LF_KFE: axis 0 1 0 -> 1 0 0; child LF_shank -> LF_SHANK; limit lower=-2.7227 upper=-0.83776 effort=45.43 velocity=15.70 -> lower=-9.42477796076938 upper=9.42477796076938 effort=80.0 velocity=8.5; origin xyz=0 0 -0.213 rpy=0 0 0 -> xyz=0 0 0 rpy=0 0 0; parent LF_thigh -> LF_KFE_drive
- joint LH_HAA: axis 1 0 0 -> -1 0 0; child LH_hip -> LH_HIP; limit lower=-1.0472 upper=1.0472 effort=23.7 velocity=30.1 -> lower=-0.7853985 upper=0.6108655 effort=80.0 velocity=8.5; origin xyz=-0.1934 0.0465 0 rpy=0 0 0 -> xyz=0 0 0 rpy=0 0 0; parent base -> LH_HAA_drive
- joint LH_HFE: axis 0 1 0 -> -1 0 0; child LH_thigh -> LH_THIGH; limit lower=-0.5236 upper=4.5379 effort=23.7 velocity=30.1 -> lower=-9.42477796076938 upper=9.42477796076938 effort=80.0 velocity=8.5; origin xyz=0 0.0955 0 rpy=0 0 0 -> xyz=0 0 0 rpy=0 0 0; parent LH_hip -> LH_HFE_output
- joint LH_KFE: axis 0 1 0 -> 1 0 0; child LH_shank -> LH_SHANK; limit lower=-2.7227 upper=-0.83776 effort=45.43 velocity=15.70 -> lower=-9.42477796076938 upper=9.42477796076938 effort=80.0 velocity=8.5; origin xyz=0 0 -0.213 rpy=0 0 0 -> xyz=0 0 0 rpy=0 0 0; parent LH_thigh -> LH_KFE_drive
- joint RF_HAA: child RF_hip -> RF_HIP; limit lower=-1.0472 upper=1.0472 effort=23.7 velocity=30.1 -> lower=-0.6108655 upper=0.7853985 effort=80.0 velocity=8.5; origin xyz=0.1934 -0.0465 0 rpy=0 0 0 -> xyz=0 0 0 rpy=0 0 0; parent base -> RF_HAA_drive
- joint RF_HFE: axis 0 1 0 -> 1 0 0; child RF_thigh -> RF_THIGH; limit lower=-1.5708 upper=3.4907 effort=23.7 velocity=30.1 -> lower=-9.42477796076938 upper=9.42477796076938 effort=80.0 velocity=8.5; origin xyz=0 -0.0955 0 rpy=0 0 0 -> xyz=0 0 0 rpy=0 0 0; parent RF_hip -> RF_HFE_output
- joint RF_KFE: axis 0 1 0 -> -1 0 0; child RF_shank -> RF_SHANK; limit lower=-2.7227 upper=-0.83776 effort=45.43 velocity=15.70 -> lower=-9.42477796076938 upper=9.42477796076938 effort=80.0 velocity=8.5; origin xyz=0 0 -0.213 rpy=0 0 0 -> xyz=0 0 0 rpy=0 0 0; parent RF_thigh -> RF_KFE_drive
- joint RH_HAA: axis 1 0 0 -> -1 0 0; child RH_hip -> RH_HIP; limit lower=-1.0472 upper=1.0472 effort=23.7 velocity=30.1 -> lower=-0.6108655 upper=0.7853985 effort=80.0 velocity=8.5; origin xyz=-0.1934 -0.0465 0 rpy=0 0 0 -> xyz=0 0 0 rpy=0 0 0; parent base -> RH_HAA_drive
- joint RH_HFE: axis 0 1 0 -> 1 0 0; child RH_thigh -> RH_THIGH; limit lower=-0.5236 upper=4.5379 effort=23.7 velocity=30.1 -> lower=-9.42477796076938 upper=9.42477796076938 effort=80.0 velocity=8.5; origin xyz=0 -0.0955 0 rpy=0 0 0 -> xyz=0 0 0 rpy=0 0 0; parent RH_hip -> RH_HFE_output
- joint RH_KFE: axis 0 1 0 -> -1 0 0; child RH_shank -> RH_SHANK; limit lower=-2.7227 upper=-0.83776 effort=45.43 velocity=15.70 -> lower=-9.42477796076938 upper=9.42477796076938 effort=80.0 velocity=8.5; origin xyz=0 0 -0.213 rpy=0 0 0 -> xyz=0 0 0 rpy=0 0 0; parent RH_thigh -> RH_KFE_drive

Commit message: moved meshes over to go2

File: resources/go2/urdf/go2.urdf (robot description, URDF)
Before this commit: robot anymal, 87 links, 86 joints
Links:
- link LF_FOOT: geometry collision cylinder length=0.39572 radius=0.0175; collision sphere radius=0.031455
- link LF_HAA_drive: geometry visual mesh filename=package://ocs2_robotic_assets/resources/go2/meshes/drive.dae scale=1.0 1.0 1.0
- link LF_HFE_drive: geometry collision cylinder length=0.119 radius=0.05375; visual mesh filename=package://ocs2_robotic_assets/resources/go2/meshes/drive.dae scale=1.0 1.0 1.0
- link LF_KFE_drive: geometry collision cylinder length=0.119 radius=0.05375; visual mesh filename=package://ocs2_robotic_assets/resources/go2/meshes/drive.dae scale=1.0 1.0 1.0
- link LF_hip_fixed: geometry visual mesh filename=package://ocs2_robotic_assets/resources/go2/meshes/hip.dae scale=1.0 1.0 1.0
- link LF_shank_fixed: geometry collision box size=0.13283 0.08302 0.05732; collision cylinder length=0.05732 radius=0.071
- link LF_thigh_fixed: geometry collision box size=0.093 0.063 0.285; collision cylinder length=0.08313000000000001 radius=0.07
- link LH_FOOT: geometry collision cylinder length=0.39572 radius=0.0175; collision sphere radius=0.031455
- link LH_HAA_drive: geometry visual mesh filename=package://ocs2_robotic_assets/resources/go2/meshes/drive.dae scale=1.0 1.0 1.0
- link LH_HFE_drive: geometry collision cylinder length=0.119 radius=0.05375; visual mesh filename=package://ocs2_robotic_assets/resources/go2/meshes/drive.dae scale=1.0 1.0 1.0
- link LH_KFE_drive: geometry collision cylinder length=0.119 radius=0.05375; visual mesh filename=package://ocs2_robotic_assets/resources/go2/meshes/drive.dae scale=1.0 1.0 1.0
- link LH_hip_fixed: geometry visual mesh filename=package://ocs2_robotic_assets/resources/go2/meshes/hip.dae scale=1.0 1.0 1.0
- link LH_shank_fixed: geometry collision box size=0.13283 0.08302 0.05732; collision cylinder length=0.05732 radius=0.071
- link LH_thigh_fixed: geometry collision box size=0.093 0.063 0.285; collision cylinder length=0.08313000000000001 radius=0.07
- link RF_FOOT: geometry collision cylinder length=0.39572 radius=0.0175; collision sphere radius=0.031455
- link RF_HAA_drive: geometry visual mesh filename=package://ocs2_robotic_assets/resources/go2/meshes/drive.dae scale=1.0 1.0 1.0
- link RF_HFE_drive: geometry collision cylinder length=0.119 radius=0.05375; visual mesh filename=package://ocs2_robotic_assets/resources/go2/meshes/drive.dae scale=1.0 1.0 1.0
- link RF_KFE_drive: geometry collision cylinder length=0.119 radius=0.05375; visual mesh filename=package://ocs2_robotic_assets/resources/go2/meshes/drive.dae scale=1.0 1.0 1.0
- link RF_hip_fixed: geometry visual mesh filename=package://ocs2_robotic_assets/resources/go2/meshes/hip.dae scale=1.0 1.0 1.0
- link RF_shank_fixed: geometry collision box size=0.13283 0.08302 0.05732; collision cylinder length=0.05732 radius=0.071
- link RF_thigh_fixed: geometry collision box size=0.093 0.063 0.285; collision cylinder length=0.08313000000000001 radius=0.07
- link RH_FOOT: geometry collision cylinder length=0.39572 radius=0.0175; collision sphere radius=0.031455
- link RH_HAA_drive: geometry visual mesh filename=package://ocs2_robotic_assets/resources/go2/meshes/drive.dae scale=1.0 1.0 1.0
- link RH_HFE_drive: geometry collision cylinder length=0.119 radius=0.05375; visual mesh filename=package://ocs2_robotic_assets/resources/go2/meshes/drive.dae scale=1.0 1.0 1.0
- link RH_KFE_drive: geometry collision cylinder length=0.119 radius=0.05375; visual mesh filename=package://ocs2_robotic_assets/resources/go2/meshes/drive.dae scale=1.0 1.0 1.0
- link RH_hip_fixed: geometry visual mesh filename=package://ocs2_robotic_assets/resources/go2/meshes/hip.dae scale=1.0 1.0 1.0
- link RH_shank_fixed: geometry collision box size=0.13283 0.08302 0.05732; collision cylinder length=0.05732 radius=0.071
- link RH_thigh_fixed: geometry collision box size=0.093 0.063 0.285; collision cylinder length=0.08313000000000001 radius=0.07
- link base: geometry collision box size=0.894 0.1615 0.256; collision cylinder length=0.1482 radius=0.089
- link battery: geometry visual mesh filename=package://ocs2_robotic_assets/resources/go2/meshes/battery.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 scale=1.0 1.0 1.0
- link bottom_shell: geometry visual mesh filename=package://ocs2_robotic_assets/resources/go2/meshes/bottom_s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 scale=1.0 1.0 1.0
- link docking_socket: geometry visual mesh filename=package://ocs2_robotic_assets/resources/go2/meshes/docking_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 scale=1.0 1.0 1.0
- link face_shell_front: geometry visual mesh filename=package://ocs2_robotic_assets/resources/go2/meshes/face_she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 scale=1.0 1.0 1.0
- link face_shell_rear: geometry visual mesh filename=package://ocs2_robotic_assets/resources/go2/meshes/face_she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 scale=1.0 1.0 1.0
- link lidar: geometry collision cylinder length=0.1355 radius=0.07; visual mesh filename=package://ocs2_robotic_assets/resources/go2/meshes/lidar.dae
- link top_shell: geometry visual mesh filename=package://ocs2_robotic_assets/resources/go2/meshes/top_shel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 scale=1.0 1.0 1.0

Commit message: removing unnecessary links

File: resources/go2/urdf/go2.urdf (robot description, URDF)
Before this commit: robot anymal, 87 links, 86 joints
Links:
- removed link base_inertia
- removed link body_top
- removed link top_shell
- link base: mass None -> 6.921; geometry collision box size=0.3762 0.0935 0.114; visual mesh filename=package://ocs2_robotic_assets/resources/go2/dae/base.dae
Joints:
- removed joint base_to_base_inertia
- removed joint base_to_body_top
- removed joint base_top_shell

Commit message: removing non-leg links (not including cameras)

File: resources/go2/urdf/go2.urdf (robot description, URDF)
Before this commit: robot anymal, 84 links, 83 joints
Links:
- removed link battery
- removed link bottom_shell
- removed link docking_socket
- removed link hbc_receiver
- removed link lidar
- removed link lidar_parent
Joints:
- removed joint base_battery
- removed joint base_bottom_shell
- removed joint base_hbc_receiver
- removed joint base_to_docking_socket
- removed joint base_to_lidar_parent
- removed joint lidar_parent_to_lidar

Commit message: removed rear and left cameras

File: resources/go2/urdf/go2.urdf (robot description, URDF)
Before this commit: robot anymal, 78 links, 77 joints
Links:
- removed link depth_camera_left_camera
- removed link depth_camera_left_camera_parent
- removed link depth_camera_left_depth_frame
- removed link depth_camera_left_depth_optical_frame
- removed link depth_camera_rear_lower_camera
- removed link depth_camera_rear_lower_camera_parent
- removed link depth_camera_rear_lower_depth_frame
- removed link depth_camera_rear_lower_depth_optical_frame
- removed link depth_camera_rear_upper_camera
- removed link depth_camera_rear_upper_camera_parent
- removed link depth_camera_rear_upper_depth_frame
- removed link depth_camera_rear_upper_depth_optical_frame
- removed link wide_angle_camera_rear_camera
- removed link wide_angle_camera_rear_camera_parent
Joints:
- removed joint base_to_depth_camera_left_camera
- removed joint depth_camera_left_camera_depth_to_depth_optical_frame
- removed joint depth_camera_left_camera_parent_to_depth_frame
- removed joint depth_camera_left_camera_to_camera_parent
- removed joint depth_camera_rear_lower_camera_depth_to_depth_optical_frame
- removed joint depth_camera_rear_lower_camera_parent_to_depth_frame
- removed joint depth_camera_rear_lower_camera_to_camera_parent
- removed joint depth_camera_rear_upper_camera_depth_to_depth_optical_frame
- removed joint depth_camera_rear_upper_camera_parent_to_depth_frame
- removed joint depth_camera_rear_upper_camera_to_camera_parent
- removed joint face_rear_to_depth_camera_rear_lower_camera
- removed joint face_rear_to_depth_camera_rear_upper_camera
- removed joint face_rear_to_wide_angle_camera_rear_camera
- removed joint wide_angle_camera_rear_camera_to_camera_parent
