Commit message: only running front camera

File: resources/go2/urdf/go2.urdf (robot description, URDF)
Before this commit: robot anymal, 64 links, 63 joints
Links:
- removed link depth_camera_right_camera
- removed link depth_camera_right_camera_parent
- removed link depth_camera_right_depth_frame
- removed link depth_camera_right_depth_optical_frame
- removed link face_rear
- removed link face_shell_front
- removed link face_shell_rear
Joints:
- removed joint base_face_rear
- removed joint base_face_shell_front
- removed joint base_face_shell_rear
- removed joint base_to_depth_camera_right_camera
- removed joint depth_camera_right_camera_depth_to_depth_optical_frame
- removed joint depth_camera_right_camera_parent_to_depth_frame
- removed joint depth_camera_right_camera_to_camera_parent
- joint base_face_front: origin xyz=0.4087 0 0.0205 rpy=0 0 -0.0 -> xyz=0.2 0 0.0205 rpy=0 0.0 -0.0

Commit message: can visualize a single leg (incorrectly)

File: resources/go2/urdf/go2.urdf (robot description, URDF)
Before this commit: robot anymal, 57 links, 56 joints
Links:
- removed link imu_link
- link LF_FOOT: mass 0.29644 -> 0.04; geometry collision sphere radius=0.022; visual mesh filename=package://ocs2_robotic_assets/resources/go2/dae/foot.dae
- link LF_HAA_drive: mass 2.01511 -> 0.001; geometry visual sphere radius=0.0000001
- link LF_HFE_drive: mass 2.01511 -> 0.0000001; geometry collision sphere radius=0.0000001; visual sphere radius=0.0000001
- link LF_HIP: mass 0.001 -> 0.678; geometry collision cylinder length=0.04 radius=0.046; visual mesh filename=package://ocs2_robotic_assets/resources/go2/dae/hip.dae
- link LF_KFE_drive: mass 2.01511 -> 0.001; geometry collision sphere radius=0.0000001; visual sphere radius=0.0000001
- link LF_SHANK: mass 0.001 -> 0.154; geometry collision cylinder length=0.12 radius=0.012; visual mesh filename=package://ocs2_robotic_assets/resources/go2/dae/calf.dae
- link LF_THIGH: mass 0.001 -> 1.152; geometry collision box size=0.213 0.0245 0.034; visual mesh filename=package://ocs2_robotic_assets/resources/go2/dae/thigh.dae
- link LF_hip_fixed: mass 0.36386 -> 0.001; geometry visual sphere radius=0.0000001
- link LF_thigh_fixed: mass 1.10098 -> 0.001; geometry collision sphere radius=0.0000001; collision sphere radius=0.0000001
Joints:
- removed joint imu_joint
- joint LF_HAA: limit lower=-0.7853985 upper=0.6108655 effort=80.0 velocity=8.5 -> lower=-1.0472 upper=1.0472 effort=23.7 velocity=30.1; origin xyz=0 0 0 rpy=0 0 0 -> xyz=0.1934 0.0465 0 rpy=0 0 0
- joint LF_HFE: axis -1 0 0 -> 0 1 0; limit lower=-9.42477796076938 upper=9.42477796076938 effort=80.0 velocity=8.5 -> lower=-1.5708 upper=3.4907 effort=23.7 velocity=30.1; origin xyz=0 0 0 rpy=0 0 0 -> xyz=0 0.0955 0 rpy=0 0 0
- joint LF_HFE_drive_LF_thigh_fixed: origin xyz=0 0 0 rpy=0 0 1.5707963267948966 -> xyz=0 0 0 rpy=0 0 0.0
- joint LF_KFE: axis 1 0 0 -> 0 1 0; limit lower=-9.42477796076938 upper=9.42477796076938 effort=80.0 velocity=8.5 -> lower=-2.7227 upper=-0.83776 effort=45.43 velocity=15.70; origin xyz=0 0 0 rpy=0 0 0 -> xyz=0 0 -0.213 rpy=0 0 0
- joint LF_hip_fixed_LF_HFE_output: origin xyz=0.069 0.006 0.0 rpy=0 0 -1.5707963267948966 -> xyz=0.0 0.0 0.0 rpy=0.0 0.0 0.0
- joint LF_thigh_fixed_LF_KFE_drive: origin xyz=0.0 0.1805 -0.285 rpy=0 0 1.5707963267948966 -> xyz=0.0 0.0 0.0 rpy=0 0 0.0
- joint base_LF_HAA_drive: origin xyz=0.304 0.109 0.0 rpy=0 0 0.0 -> xyz=0.0 0.0 0.0 rpy=0 0 0.0

Commit message: FL leg works

File: resources/go2/urdf/go2.urdf (robot description, URDF)
Before this commit: robot anymal, 56 links, 55 joints
Links:
- removed link LF_HAA_drive
- removed link LF_HFE_drive
- removed link LF_HFE_output
- removed link LF_KFE_drive
- removed link LF_hip_fixed
- removed link LF_shank_fixed
- removed link LF_thigh_fixed
- added link FL_calflower; collision cylinder length=0.065 radius=0.011
- added link FL_calflower1; collision cylinder length=0.03 radius=0.0155
Joints:
- removed joint LF_HFE_drive_LF_thigh_fixed
- removed joint LF_HIP_LF_hip_fixed
- removed joint LF_THIGH_to_LF_HFE_drive
- removed joint LF_hip_fixed_LF_HFE_output
- removed joint LF_shank_LF_shank_fixed
- removed joint LF_shank_fixed_LF_FOOT
- removed joint LF_thigh_fixed_LF_KFE_drive
- removed joint base_LF_HAA_drive
- added joint FL_calflower1_joint: type fixed, parent FL_calflower, child FL_calflower1, origin xyz=-0.01 0 -0.04 rpy=0 0.48 0, axis 0 0 0
- added joint FL_calflower_joint: type fixed, parent LF_SHANK, child FL_calflower, origin xyz=0.020 0 -0.148 rpy=0 0.05 0, axis 0 0 0
- added joint FL_foot_joint: type fixed, parent LF_SHANK, child LF_FOOT, origin xyz=0 0 -0.213 rpy=0 0 0, axis 0 0 0
- joint LF_HAA: origin xyz=0 0 0 rpy=0 0 0 -> xyz=0.1934 0.0465 0 rpy=0 0 0; parent LF_HAA_drive -> base
- joint LF_HFE: parent LF_HFE_output -> LF_HIP
- joint LF_KFE: parent LF_KFE_drive -> LF_THIGH

Commit message: added front right leg

File: resources/go2/urdf/go2.urdf (robot description, URDF)
Before this commit: robot anymal, 51 links, 50 joints
Links:
- removed link FL_calflower
- removed link FL_calflower1
- removed link RF_HAA_drive
- removed link RF_HFE_drive
- removed link RF_HFE_output
- removed link RF_KFE_drive
- removed link RF_hip_fixed
- removed link RF_shank_fixed
- removed link RF_thigh_fixed
- added link LF_calflower; collision cylinder length=0.065 radius=0.011
- added link LF_calflower1; collision cylinder length=0.03 radius=0.0155
- added link RF_calflower; collision cylinder length=0.065 radius=0.011
- added link RF_calflower1; collision cylinder length=0.03 radius=0.0155
- link RF_FOOT: mass 0.29644 -> 0.04; geometry collision sphere radius=0.022; visual mesh filename=package://ocs2_robotic_assets/resources/go2/dae/foot.dae
- link RF_HIP: mass 0.001 -> 0.678; geometry collision cylinder length=0.04 radius=0.046; visual mesh filename=package://ocs2_robotic_assets/resources/go2/dae/hip.dae
- link RF_SHANK: mass 0.001 -> 0.154; geometry collision cylinder length=0.12 radius=0.013; visual mesh filename=package://ocs2_robotic_assets/resources/go2/dae/calf_mirror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
- link RF_THIGH: mass 0.001 -> 1.152; geometry collision box size=0.213 0.0245 0.034; visual mesh filename=package://ocs2_robotic_assets/resources/go2/dae/thigh_mirro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
Joints:
- removed joint FL_calflower1_joint
- removed joint FL_calflower_joint
- removed joint FL_foot_joint
- removed joint RF_HFE_drive_RF_thigh_fixed
- removed joint RF_HIP_RF_hip_fixed
- removed joint RF_THIGH_to_RF_HFE_drive
- removed joint RF_hip_fixed_RF_HFE_output
- removed joint RF_shank_RF_shank_fixed
- removed joint RF_shank_fixed_RF_FOOT
- removed joint RF_thigh_fixed_RF_KFE_drive
- removed joint base_RF_HAA_drive
- added joint LF_calflower1_joint: type fixed, parent LF_calflower, child LF_calflower1, origin xyz=-0.01 0 -0.04 rpy=0 0.48 0, axis 0 0 0
- added joint LF_calflower_joint: type fixed, parent LF_SHANK, child LF_calflower, origin xyz=0.020 0 -0.148 rpy=0 0.05 0, axis 0 0 0
- added joint LF_foot_joint: type fixed, parent LF_SHANK, child LF_FOOT, origin xyz=0 0 -0.213 rpy=0 0 0, axis 0 0 0
- added joint RF_calflower1_joint: type fixed, parent RF_calflower, child RF_calflower1, origin xyz=-0.01 0 -0.04 rpy=0 0.48 0, axis 0 0 0
- added joint RF_calflower_joint: type fixed, parent RF_SHANK, child RF_calflower, origin xyz=0.020 0 -0.148 rpy=0 0.05 0, axis 0 0 0
- added joint RF_foot_joint: type fixed, parent RF_SHANK, child RF_FOOT, origin xyz=0 0 -0.213 rpy=0 0 0, axis 0 0 0
- joint RF_HAA: limit lower=-0.6108655 upper=0.7853985 effort=80.0 velocity=8.5 -> lower=-1.0472 upper=1.0472 effort=23.7 velocity=30.1; origin xyz=0 0 0 rpy=0 0 0 -> xyz=0.1934 -0.0465 0 rpy=0 0 0; parent RF_HAA_drive -> base
- joint RF_HFE: axis 1 0 0 -> 0 1 0; limit lower=-9.42477796076938 upper=9.42477796076938 effort=80.0 velocity=8.5 -> lower=-1.5708 upper=3.4907 effort=23.7 velocity=30.1; origin xyz=0 0 0 rpy=0 0 0 -> xyz=0 -0.0955 0 rpy=0 0 0; parent RF_HFE_output -> RF_HIP
- joint RF_KFE: axis -1 0 0 -> 0 1 0; limit lower=-9.42477796076938 upper=9.42477796076938 effort=80.0 velocity=8.5 -> lower=-2.7227 upper=-0.83776 effort=45.43 velocity=15.70; origin xyz=0 0 0 rpy=0 0 0 -> xyz=0 0 -0.213 rpy=0 0 0; parent RF_KFE_drive -> RF_THIGH

Commit message: adding rear left leg

File: resources/go2/urdf/go2.urdf (robot description, URDF)
Before this commit: robot anymal, 46 links, 45 joints
Links:
- removed link LH_HAA_drive
- removed link LH_HFE_drive
- removed link LH_HFE_output
- removed link LH_KFE_drive
- removed link LH_hip_fixed
- removed link LH_shank_fixed
- removed link LH_thigh_fixed
- added link LH_calflower; collision cylinder length=0.065 radius=0.011
- added link LH_calflower1; collision cylinder length=0.03 radius=0.0155
- link LH_FOOT: mass 0.29644 -> 0.04; geometry collision sphere radius=0.022; visual mesh filename=package://ocs2_robotic_assets/resources/go2/dae/foot.dae
- link LH_HIP: mass 0.001 -> 0.678; geometry collision cylinder length=0.04 radius=0.046; visual mesh filename=package://ocs2_robotic_assets/resources/go2/dae/hip.dae
- link LH_SHANK: mass 0.001 -> 0.154; geometry collision cylinder length=0.12 radius=0.013; visual mesh filename=package://ocs2_robotic_assets/resources/go2/dae/calf.dae
- link LH_THIGH: mass 0.001 -> 1.152; geometry collision box size=0.213 0.0245 0.034; visual mesh filename=package://ocs2_robotic_assets/resources/go2/dae/thigh.dae
Joints:
- removed joint LH_HFE_drive_LH_thigh_fixed
- removed joint LH_HIP_LH_hip_fixed
- removed joint LH_THIGH_to_LH_HFE_drive
- removed joint LH_hip_fixed_LH_HFE_output
- removed joint LH_shank_LH_shank_fixed
- removed joint LH_shank_fixed_LH_FOOT
- removed joint LH_thigh_fixed_LH_KFE_drive
- removed joint base_LH_HAA_drive
- added joint LH_calflower1_joint: type fixed, parent LH_calflower, child LH_calflower1, origin xyz=-0.01 0 -0.04 rpy=0 0.48 0, axis 0 0 0
- added joint LH_calflower_joint: type fixed, parent LH_SHANK, child LH_calflower, origin xyz=0.020 0 -0.148 rpy=0 0.05 0, axis 0 0 0
- added joint LH_foot_joint: type fixed, parent LH_SHANK, child LH_FOOT, origin xyz=0 0 -0.213 rpy=0 0 0, axis 0 0 0
- joint LH_HAA: axis -1 0 0 -> 1 0 0; limit lower=-0.7853985 upper=0.6108655 effort=80.0 velocity=8.5 -> lower=-1.0472 upper=1.0472 effort=23.7 velocity=30.1; origin xyz=0 0 0 rpy=0 0 0 -> xyz=-0.1934 0.0465 0 rpy=0 0 0; parent LH_HAA_drive -> base
- joint LH_HFE: axis -1 0 0 -> 0 1 0; limit lower=-9.42477796076938 upper=9.42477796076938 effort=80.0 velocity=8.5 -> lower=-0.5236 upper=4.5379 effort=23.7 velocity=30.1; origin xyz=0 0 0 rpy=0 0 0 -> xyz=0 0.0955 0 rpy=0 0 0; parent LH_HFE_output -> LH_HIP
- joint LH_KFE: axis 1 0 0 -> 0 1 0; limit lower=-9.42477796076938 upper=9.42477796076938 effort=80.0 velocity=8.5 -> lower=-2.7227 upper=-0.83776 effort=45.43 velocity=15.70; origin xyz=0 0 0 rpy=0 0 0 -> xyz=0 0 -0.213 rpy=0 0 0; parent LH_KFE_drive -> LH_THIGH

Commit message: added rear right leg

File: resources/go2/urdf/go2.urdf (robot description, URDF)
Before this commit: robot anymal, 41 links, 40 joints
Links:
- removed link RH_HAA_drive
- removed link RH_HFE_drive
- removed link RH_HFE_output
- removed link RH_KFE_drive
- removed link RH_hip_fixed
- removed link RH_shank_fixed
- removed link RH_thigh_fixed
- added link RH_calflower; collision cylinder length=0.065 radius=0.011
- added link RH_calflower1; collision cylinder length=0.03 radius=0.0155
- link RH_FOOT: mass 0.29644 -> 0.04; geometry collision sphere radius=0.022; visual mesh filename=package://ocs2_robotic_assets/resources/go2/dae/foot.dae
- link RH_HIP: mass 0.001 -> 0.678; geometry collision cylinder length=0.04 radius=0.046; visual mesh filename=package://ocs2_robotic_assets/resources/go2/dae/hip.dae
- link RH_SHANK: mass 0.001 -> 0.154; geometry collision cylinder length=0.12 radius=0.013; visual mesh filename=package://ocs2_robotic_assets/resources/go2/dae/calf_mirror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
- link RH_THIGH: mass 0.001 -> 1.152; geometry collision box size=0.213 0.0245 0.034; visual mesh filename=package://ocs2_robotic_assets/resources/go2/dae/thigh_mirro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
Joints:
- removed joint RH_HFE_drive_RH_thigh_fixed
- removed joint RH_HIP_RH_hip_fixed
- removed joint RH_THIGH_to_RH_HFE_drive
- removed joint RH_hip_fixed_RH_HFE_output
- removed joint RH_shank_RH_shank_fixed
- removed joint RH_shank_fixed_RH_FOOT
- removed joint RH_thigh_fixed_RH_KFE_drive
- removed joint base_RH_HAA_drive
- added joint RH_calflower1_joint: type fixed, parent RH_calflower, child RH_calflower1, origin xyz=-0.01 0 -0.04 rpy=0 0.48 0, axis 0 0 0
- added joint RH_calflower_joint: type fixed, parent RH_SHANK, child RH_calflower, origin xyz=0.020 0 -0.148 rpy=0 0.05 0, axis 0 0 0
- added joint RH_foot_joint: type fixed, parent RH_SHANK, child RH_FOOT, origin xyz=0 0 -0.213 rpy=0 0 0, axis 0 0 0
- joint RH_HAA: axis -1 0 0 -> 1 0 0; limit lower=-0.6108655 upper=0.7853985 effort=80.0 velocity=8.5 -> lower=-1.0472 upper=1.0472 effort=23.7 velocity=30.1; origin xyz=0 0 0 rpy=0 0 0 -> xyz=-0.1934 -0.0465 0 rpy=0 0 0; parent RH_HAA_drive -> base
- joint RH_HFE: axis 1 0 0 -> 0 1 0; limit lower=-9.42477796076938 upper=9.42477796076938 effort=80.0 velocity=8.5 -> lower=-0.5236 upper=4.5379 effort=23.7 velocity=30.1; origin xyz=0 0 0 rpy=0 0 0 -> xyz=0 -0.0955 0 rpy=0 0 0; parent RH_HFE_output -> RH_HIP
- joint RH_KFE: axis -1 0 0 -> 0 1 0; limit lower=-9.42477796076938 upper=9.42477796076938 effort=80.0 velocity=8.5 -> lower=-2.7227 upper=-0.83776 effort=45.43 velocity=15.70; origin xyz=0 0 0 rpy=0 0 0 -> xyz=0 0 -0.213 rpy=0 0 0; parent RH_KFE_drive -> RH_THIGH

Commit message: trimmed more unnecessary links/joints

File: resources/go2/urdf/go2.urdf (robot description, URDF)
Before this commit: robot anymal, 36 links, 35 joints
Links:
- removed link depth_camera_front_lower_camera
- removed link depth_camera_front_lower_camera_parent
- removed link depth_camera_front_lower_depth_frame
- removed link depth_camera_front_lower_depth_optical_frame
- removed link depth_camera_front_upper_camera
- removed link depth_camera_front_upper_camera_parent
- removed link depth_camera_front_upper_depth_frame
- removed link depth_camera_front_upper_depth_optical_frame
- removed link face_front
- removed link wide_angle_camera_front_camera
- removed link wide_angle_camera_front_camera_parent
- added link base_inertia, mass 6.921
- link base: mass 6.921 -> None
Joints:
- removed joint base_face_front
- removed joint depth_camera_front_lower_camera_depth_to_depth_optical_frame
- removed joint depth_camera_front_lower_camera_parent_to_depth_frame
- removed joint depth_camera_front_lower_camera_to_camera_parent
- removed joint depth_camera_front_upper_camera_depth_to_depth_optical_frame
- removed joint depth_camera_front_upper_camera_parent_to_depth_frame
- removed joint depth_camera_front_upper_camera_to_camera_parent
- removed joint face_front_to_depth_camera_front_lower_camera
- removed joint face_front_to_depth_camera_front_upper_camera
- removed joint face_front_to_wide_angle_camera_front_camera
- removed joint wide_angle_camera_front_camera_to_camera_parent
- added joint base_to_base_inertia: type fixed, parent base, child base_inertia, origin xyz=0 0 0 rpy=0 0 0

Commit message: kill me

File: resources/go2/urdf/go2.urdf (robot description, URDF)
Before this commit: robot anymal, 26 links, 25 joints
Links:
- removed link base_inertia
- added link Head_lower, mass 0.001; collision sphere radius=0.047
- added link Head_upper, mass 0.001; collision cylinder length=0.09 radius=0.05
- link base: mass None -> 6.921
Joints:
- removed joint base_to_base_inertia
- added joint Head_lower_joint: type fixed, parent Head_upper, child Head_lower, origin xyz=0.008 0 -0.07 rpy=0 0 0, axis 0 0 0
- added joint Head_upper_joint: type fixed, parent base, child Head_upper, origin xyz=0.285 0 0.01 rpy=0 0 0, axis 0 0 0
